Commit message: add dummy camera and dummy imu

File: urdf/falcon.urdf.xacro (robot description, xacro)
@@ -15,4 +15,5 @@
   <xacro:property name="chassis_width" value="0.73"/>
   <xacro:property name="chassis_length" value="1.23"/>
+  <xacro:property name="imu_size" value="0.1"/>
   <!-- TODO: measure these -->
   <xacro:property name="wheel_base" value="0.505"/>
@@ -86,5 +87,5 @@
           <mesh filename="package://falcon_description/meshes/visual/chassis.dae"/>
       </geometry>
-      <material name="red"/>
+      <material name="light_grey"/>
     </visual>
     <collision>
@@ -100,4 +101,70 @@
     </inertial>
   </link>
+  <link name="imu_link">
+    <visual>
+      <origin xyz="0 0 0"/>
+		<geometry>
+      	  <box size="${imu_size} ${imu_size} ${imu_size}"/>
+      	</geometry>
+      <material name="green"/>
+    </visual>
+    <inertial>
+      <mass value="0.001"/>
+      <origin xyz="0 0 0" rpy="0 0 0"/>
+      <inertia ixx="${dummy_inertia}" ixy="0.0" ixz="0.0" iyy="${dummy_inertia}" iyz="0.0" izz="${dummy_inertia}"/>
+    </inertial>
+  </link>
+  <joint name="imu_joint" type="fixed">
+    <parent link="chassis"/>
+    <child link="imu_link"/>
+  </joint>
+  <link name="ZED_left_camera">
+        <visual>
+            <origin xyz="0 0 0" rpy="0 1.57 0"/>
+            <geometry>
+                <cylinder radius="0.007" length=".031"/>
+            </geometry>
+            <material name="dark_grey">
+                <color rgba="0.1 0.1 0.1 1"/>
+            </material>
+        </visual>
+    </link>
+    <link name="ZED_center">
+        <visual>
+            <origin xyz="0 0 0" rpy="0 0 0"/>
+            <geometry>
+                <mesh filename="package://amee_description/urdf/ZED.stl" />
+            </geometry>
+            <material name="light_grey">
+                <color rgba="0.8 0.8 0.8 0.8"/>
+            </material>
+        </visual>
+    </link>
+    <link name="ZED_right_camera">
+        <visual>
+            <origin xyz="0 0 0" rpy="0 1.57 0"/>
+            <geometry>
+                <cylinder radius="0.007" length=".031"/>
+            </geometry>
+            <material name="dark_grey">
+                <color rgba="0.1 0.1 0.1 1"/>
+            </material>
+        </visual>
+    </link>
+    <joint name="ZED_center_joint" type="fixed">
+        <parent link="ZED_left_camera"/>
+        <child link="ZED_center"/>
+        <origin xyz="0 -0.06 0" rpy="0 0 0" />
+    </joint>
+    <joint name="ZED_right_camera_joint" type="fixed">
+        <parent link="ZED_left_camera"/>
+        <child link="ZED_right_camera"/>
+        <origin xyz="0 -0.12 0" rpy="0 0 0" />
+    </joint>
+  <joint name="zed_joint" type="fixed">
+    <parent link="chassis"/>
+    <child link="ZED_left_camera"/>
+	<origin rpy="0 0 ${pi}" xyz="${-chassis_length/2} -0.06 0.0"/>
+  </joint>
   <xacro:wheel prefix="left_front" reflect="1">
 	  <origin xyz="${wheel_base/2} ${wheel_track/2} ${wheel_z_offset}" rpy="0 0 0"/>
